Commit message: Define M_PI $(find turtlebot3_description)/urdf/common_properties.xacro defined M_PI But, It was deleted from upstream : https://github.com/ROBOTIS-GIT/turtlebot3/commit/76ab4240eac7ae4877f30d51e8dbe51c04387d77#diff-a6a880b297e353a2b2fc851cb9514b97

File: urdf/turtlebot3_burger_stereo.urdf.xacro (robot description, xacro)
@@ -3,4 +3,5 @@
   <xacro:include filename="$(find turtlebot3_description)/urdf/common_properties.xacro"/>
   <xacro:include filename="$(find turtlebot3_stereo_description)/urdf/turtlebot3_burger_stereo.gazebo.xacro"/>
+  <xacro:property name="M_PI" value="3.1415926535897931" />
   <link name="base_footprint"/>
   <joint name="base_joint" type="fixed">
